Commit message: add nav_link in urdf

File: whud_slam/config/whud.urdf (robot description, URDF)
Before this commit: robot whud, 3 links, 2 joints
Links:
- added link nav_link
Joints:
- added joint nav_joint: type fixed, parent track_link, child nav_link, origin xyz=0.07 0 0 rpy=0 0 0

Commit message: update nav_joint

File: whud_slam/config/whud.urdf (robot description, URDF)
Before this commit: robot whud, 4 links, 3 joints
Joints:
- joint nav_joint: origin xyz=0.07 0 0 rpy=0 0 0 -> xyz=-0.07 0 0 rpy=0 0 0

Commit message: update navigation

File: whud_slam/config/whud.urdf (robot description, URDF)
Before this commit: robot whud, 4 links, 3 joints
Joints:
- joint nav_joint: origin xyz=-0.07 0 0 rpy=0 0 0 -> xyz=-0.08 0 0 rpy=0 0 0
